Commit message: Add gripper to staubli simulator

File: staubli_tx2_60_gazebo/urdf/tx2_60.xacro (robot description, xacro)
@@ -3,7 +3,11 @@
   <!-- TX60 -->
   <xacro:include filename="$(find staubli_tx2_60_gazebo)/urdf/tx2_60_macro.xacro"/>
-  <xacro:include filename="$(find staubli_tx2_60_gazebo)/urdf/asus_xtion_macro.xacro"/>
+  <xacro:include filename="$(find staubli_tx2_60_gazebo)/urdf/_d435.urdf.xacro" />
+  <xacro:include filename="$(find staubli_tx2_60_support)/urdf/gripper_macro.xacro"/>
   <xacro:staubli_tx2_60_robot prefix=""/>
-  <xacro:asus_xtion prefix=""/>
+  <xacro:gripper prefix=""/>
+  <sensor_d435 parent="link_6">
+    <origin xyz="0.105 -0.0 0.01" rpy="0 -1.57 0"/>
+  </sensor_d435>
   <!-- Fix robot to Gazebo world -->
   <link name="world"/>

File: staubli_tx2_60_support/urdf/gripper_macro.xacro (robot description, xacro)
@@ -6,5 +6,5 @@
         <parent link="link_6" />
         <child link="gripper_base_link" />
-        <origin rpy="3.14 0 0" xyz="0.0 0 0.001" />
+        <origin rpy="0 0 3.14" xyz="0.0 0 0.001" />
     </joint>
     <!-- Gripper Base -->

Commit message: towards, random pick place with staubli

File: staubli_tx2_60_gazebo/urdf/tx2_60.xacro (robot description, xacro)
@@ -8,5 +8,5 @@
   <xacro:gripper prefix=""/>
   <sensor_d435 parent="link_6">
-    <origin xyz="0.105 -0.0 0.01" rpy="0 -1.57 0"/>
+    <origin xyz="0.105 -0.0 0.01" rpy="0 -1.57 3.14"/>
   </sensor_d435>
   <!-- Fix robot to Gazebo world -->
