Commit message: TX 90 WORKS

File: staubli_tx2_90_support/urdf/tx2_90_macro.xacro (robot description, xacro)
@@ -1,118 +1,153 @@
 <?xml version="1.0"?>
 <robot xmlns:xacro="http://wiki.ros.org/xacro">
-  <xacro:include filename="$(find staubli_resources)/urdf/common_materials.xacro"/>
+  <xacro:include filename="$(find staubli_resources)/urdf/common_materials.xacro" />
   <xacro:macro name="staubli_tx2_90" params="prefix">
     <!-- links: main serial chain -->
     <link name="${prefix}base_link">
       <visual>
-        <origin xyz="0 0 0" rpy="0 0 0"/>
-        <geometry>
-          <mesh filename="package://staubli_tx2_90_support/meshes/tx2_90/visual/base_link.stl"/>
-        </geometry>
-        <xacro:material_staubli_ral_melon_yellow />
-      </visual>
-      <collision>
-        <origin xyz="0 0 0" rpy="0 0 0"/>
-        <geometry>
-          <mesh filename="package://staubli_tx2_90_support/meshes/tx2_90/collision/base_link.stl"/>
-        </geometry>
-      </collision>
+        <origin xyz="0 0 0" rpy="0 0 0" />
+        <geometry>
+          <mesh filename="package://staubli_tx2_90_support/meshes/tx2_90/visual/base_link.stl" />
+        </geometry>
+        <xacro:material_staubli_ral_melon_yellow />
+      </visual>
+      <collision>
+        <origin xyz="0 0 0" rpy="0 0 0" />
+        <geometry>
+          <mesh filename="package://staubli_tx2_90_support/meshes/tx2_90/collision/base_link.stl" />
+        </geometry>
+      </collision>
+      <inertial>
+        <mass value="10.733459" />
+        <origin xyz="0.014288 0.000001 0.122264" rpy="0.0 0.0 0.0" />
+        <inertia ixx="0.096590" ixy="-0.000005" ixz="-0.003803" iyy="0.087591" iyz="-0.000001" izz="0.081632" />
+      </inertial>
     </link>
     <link name="${prefix}link_1">
       <visual>
-        <origin xyz="0 0 0" rpy="0 0 0"/>
-        <geometry>
-          <mesh filename="package://staubli_tx2_90_support/meshes/tx2_90/visual/link_1.stl"/>
-        </geometry>
-        <xacro:material_staubli_ral_melon_yellow />
-      </visual>
-      <collision>
-        <origin xyz="0 0 0" rpy="0 0 0"/>
-        <geometry>
-          <mesh filename="package://staubli_tx2_90_support/meshes/tx2_90/collision/link_1.stl"/>
-        </geometry>
-      </collision>
+        <origin xyz="0 0 0" rpy="0 0 0" />
+        <geometry>
+          <mesh filename="package://staubli_tx2_90_support/meshes/tx2_90/visual/link_1.stl" />
+        </geometry>
+        <xacro:material_staubli_ral_melon_yellow />
+      </visual>
+      <collision>
+        <origin xyz="0 0 0" rpy="0 0 0" />
+        <geometry>
+          <mesh filename="package://staubli_tx2_90_support/meshes/tx2_90/collision/link_1.stl" />
+        </geometry>
+      </collision>
+      <inertial>
+        <mass value="16.934564" />
+        <origin xyz="0.019143 0.024764 -0.064596" rpy="0.0 0.0 0.0" />
+        <inertia ixx="0.222318" ixy="0.016499" ixz="0.023794" iyy="0.208959" iyz="0.031663" izz="0.157081" />
+      </inertial>
     </link>
     <link name="${prefix}link_2">
       <visual>
-        <origin xyz="0 0 0" rpy="0 0 0"/>
-        <geometry>
-          <mesh filename="package://staubli_tx2_90_support/meshes/tx2_90/visual/link_2.stl"/>
-        </geometry>
-        <xacro:material_staubli_ral_melon_yellow />
-      </visual>
-      <collision>
-        <origin xyz="0 0 0" rpy="0 0 0"/>
-        <geometry>
-          <mesh filename="package://staubli_tx2_90_support/meshes/tx2_90/collision/link_2.stl"/>
-        </geometry>
-      </collision>
+        <origin xyz="0 0 0" rpy="0 0 0" />
+        <geometry>
+          <mesh filename="package://staubli_tx2_90_support/meshes/tx2_90/visual/link_2.stl" />
+        </geometry>
+        <xacro:material_staubli_ral_melon_yellow />
+      </visual>
+      <collision>
+        <origin xyz="0 0 0" rpy="0 0 0" />
+        <geometry>
+          <mesh filename="package://staubli_tx2_90_support/meshes/tx2_90/collision/link_2.stl" />
+        </geometry>
+      </collision>
+      <inertial>
+        <mass value="12.98711" />
+        <origin xyz="-0.000008 0.221181 0.173052" rpy="0.0 0.0 0.0" />
+        <inertia ixx="0.425299" ixy="0.000005" ixz="-0.000004" iyy="0.452311" iyz="-0.002920" izz="0.054493" />
+      </inertial>
     </link>
     <link name="${prefix}link_3">
       <visual>
-        <origin xyz="0 0 0" rpy="0 0 0"/>
-        <geometry>
-          <mesh filename="package://staubli_tx2_90_support/meshes/tx2_90/visual/link_3.stl"/>
-        </geometry>
-        <xacro:material_staubli_ral_melon_yellow />
-      </visual>
-      <collision>
-        <origin xyz="0 0 0" rpy="0 0 0"/>
-        <geometry>
-          <mesh filename="package://staubli_tx2_90_support/meshes/tx2_90/collision/link_3.stl"/>
-        </geometry>
-      </collision>
+        <origin xyz="0 0 0" rpy="0 0 0" />
+        <geometry>
+          <mesh filename="package://staubli_tx2_90_support/meshes/tx2_90/visual/link_3.stl" />
+        </geometry>
+        <xacro:material_staubli_ral_melon_yellow />
+      </visual>
+      <collision>
+        <origin xyz="0 0 0" rpy="0 0 0" />
+        <geometry>
+          <mesh filename="package://staubli_tx2_90_support/meshes/tx2_90/collision/link_3.stl" />
+        </geometry>
+      </collision>
+      <inertial>
+        <mass value="7.50151" />
+        <origin xyz="0.000002 0.065008 0.003572" rpy="0.0 0.0 0.0" />
+        <inertia ixx="0.058902" ixy="0.000000" ixz="0.000001" iyy="0.056884" iyz="-0.003672" izz="0.034271" />
+      </inertial>
     </link>
     <link name="${prefix}link_4">
       <visual>
-        <origin xyz="0 0 0" rpy="0 0 0"/>
-        <geometry>
-          <mesh filename="package://staubli_tx2_90_support/meshes/tx2_90/visual/link_4.stl"/>
-        </geometry>
-        <xacro:material_staubli_ral_melon_yellow />
-      </visual>
-      <collision>
-        <origin xyz="0 0 0" rpy="0 0 0"/>
-        <geometry>
-          <mesh filename="package://staubli_tx2_90_support/meshes/tx2_90/collision/link_4.stl"/>
-        </geometry>
-      </collision>
+        <origin xyz="0 0 0" rpy="0 0 0" />
+        <geometry>
+          <mesh filename="package://staubli_tx2_90_support/meshes/tx2_90/visual/link_4.stl" />
+        </geometry>
+        <xacro:material_staubli_ral_melon_yellow />
+      </visual>
+      <collision>
+        <origin xyz="0 0 0" rpy="0 0 0" />
+        <geometry>
+          <mesh filename="package://staubli_tx2_90_support/meshes/tx2_90/collision/link_4.stl" />
+        </geometry>
+      </collision>
+      <inertial>
+        <mass value="4.54015" />
+        <origin xyz="-0.002488 0.049988 0.296156" rpy="0.0 0.0 0.0" />
+        <inertia ixx="0.043246" ixy="0.000003" ixz="-0.000683" iyy="0.038394" iyz="-0.000004" izz="0.014525" />
+      </inertial>
     </link>
     <link name="${prefix}link_5">
       <visual>
-        <origin xyz="0 0 0" rpy="0 0 0"/>
-        <geometry>
-          <mesh filename="package://staubli_tx2_90_support/meshes/tx2_90/visual/link_5.stl"/>
+        <origin xyz="0 0 0" rpy="0 0 0" />
+        <geometry>
+          <mesh filename="package://staubli_tx2_90_support/meshes/tx2_90/visual/link_5.stl" />
         </geometry>
         <xacro:material_staubli_ral_grey_aluminium />
       </visual>
       <collision>
-        <origin xyz="0 0 0" rpy="0 0 0"/>
-        <geometry>
-          <mesh filename="package://staubli_tx2_90_support/meshes/tx2_90/collision/link_5.stl"/>
-        </geometry>
-      </collision>
+        <origin xyz="0 0 0" rpy="0 0 0" />
+        <geometry>
+          <mesh filename="package://staubli_tx2_90_support/meshes/tx2_90/collision/link_5.stl" />
+        </geometry>
+      </collision>
+      <inertial>
+        <mass value="0.56876" />
+        <origin xyz="0.000000 0.049931 0.222823" rpy="0.0 0.0 0.0" />
+        <inertia ixx="0.001084" ixy="0.000000" ixz="0.000000" iyy="0.001123" iyz="0.000001" izz="0.000383" />
+      </inertial>
     </link>
     <link name="${prefix}link_6">
       <visual>
-        <origin xyz="0 0 0" rpy="0 0 0"/>
-        <geometry>
-          <mesh filename="package://staubli_tx2_90_support/meshes/tx2_90/visual/link_6.stl"/>
+        <origin xyz="0 0 0" rpy="0 0 0" />
+        <geometry>
+          <mesh filename="package://staubli_tx2_90_support/meshes/tx2_90/visual/link_6.stl" />
         </geometry>
         <xacro:material_staubli_ral_grey_aluminium />
       </visual>
       <collision>
-        <origin xyz="0 0 0" rpy="0 0 0"/>
-        <geometry>
-          <mesh filename="package://staubli_tx2_90_support/meshes/tx2_90/collision/link_6.stl"/>
-        </geometry>
-      </collision>
+        <origin xyz="0 0 0" rpy="0 0 0" />
+        <geometry>
+          <mesh filename="package://staubli_tx2_90_support/meshes/tx2_90/collision/link_6.stl" />
+        </geometry>
+      </collision>
+      <inertial>
+        <mass value="0.03098" />
+        <origin xyz="-0.000243 0.050000 -0.006293" rpy="0.0 0.0 0.0" />
+        <inertia ixx="0.000012" ixy="0.000000" ixz="0.000000" iyy="0.000011" iyz="0.000000" izz="0.000022" />
+      </inertial>
     </link>
     <!-- joints: main serial chain -->
     <joint name="${prefix}joint_1" type="revolute">
-      <origin xyz="0 0 0.478" rpy="0 0 0"/>
-      <parent link="${prefix}base_link"/>
-      <child link="${prefix}link_1"/>
-      <axis xyz="0 0 1"/>
+      <origin xyz="0 0 0.478" rpy="0 0 0" />
+      <parent link="${prefix}base_link" />
+      <child link="${prefix}link_1" />
+      <axis xyz="0 0 1" />
       <!-- from Staubli instruction manual:
       (1) effort limit = 318 Nm if floor mounted
@@ -122,40 +157,40 @@
     </joint>
     <joint name="${prefix}joint_2" type="revolute">
-      <origin xyz="0.050 0 0" rpy="0 0 0"/>
-      <parent link="${prefix}link_1"/>
-      <child link="${prefix}link_2"/>
-      <axis xyz="0 1 0"/>
+      <origin xyz="0.050 0 0" rpy="0 0 0" />
+      <parent link="${prefix}link_1" />
+      <child link="${prefix}link_2" />
+      <axis xyz="0 1 0" />
       <!-- nominal velocity limits are used -->
       <limit lower="${radians(-130)}" upper="${radians(147.5)}" effort="166.0" velocity="${radians(210)}" />
     </joint>
     <joint name="${prefix}joint_3" type="revolute">
-      <origin xyz="0 0.05 0.425" rpy="0 0 0"/>
-      <parent link="${prefix}link_2"/>
-      <child link="${prefix}link_3"/>
-      <axis xyz="0 1 0"/>
+      <origin xyz="0 0.05 0.425" rpy="0 0 0" />
+      <parent link="${prefix}link_2" />
+      <child link="${prefix}link_3" />
+      <axis xyz="0 1 0" />
       <!-- nominal velocity limits are used -->
       <limit lower="${radians(-145)}" upper="${radians(145)}" effort="76.0" velocity="${radians(315)}" />
     </joint>
     <joint name="${prefix}joint_4" type="revolute">
-      <origin xyz="0 0 0" rpy="0 0 0"/>
-      <parent link="${prefix}link_3"/>
-      <child link="${prefix}link_4"/>
-      <axis xyz="0 0 1"/>
+      <origin xyz="0 0 0" rpy="0 0 0" />
+      <parent link="${prefix}link_3" />
+      <child link="${prefix}link_4" />
+      <axis xyz="0 0 1" />
       <!-- nominal velocity limits are used -->
       <limit lower="${radians(-270)}" upper="${radians(270)}" effort="34.0" velocity="${radians(450)}" />
     </joint>
     <joint name="${prefix}joint_5" type="revolute">
-      <origin xyz="0 0 0.425" rpy="0 0 0"/>
-      <parent link="${prefix}link_4"/>
-      <child link="${prefix}link_5"/>
-      <axis xyz="0 1 0"/>
+      <origin xyz="0 0 0.425" rpy="0 0 0" />
+      <parent link="${prefix}link_4" />
+      <child link="${prefix}link_5" />
+      <axis xyz="0 1 0" />
       <!-- nominal velocity limits are used -->
       <limit lower="${radians(-115)}" upper="${radians(140)}" effort="29.0" velocity="${radians(370)}" />
     </joint>
     <joint name="${prefix}joint_6" type="revolute">
-      <origin xyz="0 0 0.100" rpy="0 0 0"/>
-      <parent link="${prefix}link_5"/>
-      <child link="${prefix}link_6"/>
-      <axis xyz="0 0 1"/>
+      <origin xyz="0 0 0.100" rpy="0 0 0" />
+      <parent link="${prefix}link_5" />
+      <child link="${prefix}link_6" />
+      <axis xyz="0 0 1" />
       <!-- nominal velocity limits are used -->
       <limit lower="${radians(-270)}" upper="${radians(270)}" effort="11.0" velocity="${radians(630)}" />
@@ -164,7 +199,7 @@
     <link name="${prefix}base" />
     <joint name="${prefix}base_link-base" type="fixed">
-      <origin xyz="0 0 0.478" rpy="0 0 0"/>
-      <parent link="${prefix}base_link"/>
-      <child link="${prefix}base"/>
+      <origin xyz="0 0 0.478" rpy="0 0 0" />
+      <parent link="${prefix}base_link" />
+      <child link="${prefix}base" />
     </joint>
     <!-- ROS-Industrial 'flange' frame: attachment point for EEF models -->
