Commit message: rx160 not in good shape

File: staubli_rx160_support/urdf/rx160_macro.xacro (robot description, xacro)
@@ -1,219 +1,205 @@
 <?xml version="1.0"?>
 <robot xmlns:xacro="http://wiki.ros.org/xacro">
-  <xacro:include filename="$(find staubli_resources)/urdf/common_materials.xacro"/>
+  <xacro:include filename="$(find staubli_resources)/urdf/common_materials.xacro" />
   <xacro:macro name="staubli_rx160" params="prefix">
     <!-- links: main serial chain -->
     <link name="${prefix}base_link">
       <visual>
-        <origin xyz="0 0 0" rpy="0 0 0"/>
-        <geometry>
-          <mesh filename="package://staubli_rx160_support/meshes/rx160/visual/base_link.stl"/>
-        </geometry>
-        <xacro:material_staubli_ral_melon_yellow />
-      </visual>
-      <collision>
-        <origin xyz="0 0 0" rpy="0 0 0"/>
-        <geometry>
-          <mesh filename="package://staubli_rx160_support/meshes/rx160/collision/base_link.stl"/>
-        </geometry>
-      </collision>
-      <inertial>
-          <mass value="23.085357"/>
-          <origin xyz="0.007579 0.000017 0.180670" rpy="0.0 0.0 0.0"/>
-          <inertia ixx="0.343576" ixy="-0.000062" ixz="-0.002079"
-                                  iyy="0.336217"  iyz="-0.000014"
-                                                  izz="0.334050"/>
+        <origin xyz="0 0 0" rpy="0 0 0" />
+        <geometry>
+          <mesh filename="package://staubli_rx160_support/meshes/rx160/visual/base_link.stl" />
+        </geometry>
+        <xacro:material_staubli_ral_melon_yellow />
+      </visual>
+      <collision>
+        <origin xyz="0 0 0" rpy="0 0 0" />
+        <geometry>
+          <mesh filename="package://staubli_rx160_support/meshes/rx160/collision/base_link.stl" />
+        </geometry>
+      </collision>
+      <inertial>
+        <mass value="10.733459" />
+        <origin xyz="0.014288 0.000001 0.122264" rpy="0.0 0.0 0.0" />
+        <inertia ixx="0.096590" ixy="-0.000005" ixz="-0.003803" iyy="0.087591" iyz="-0.000001" izz="0.081632" />
       </inertial>
     </link>
     <link name="${prefix}link_1">
       <visual>
-        <origin xyz="0 0 0" rpy="0 0 0"/>
-        <geometry>
-          <mesh filename="package://staubli_rx160_support/meshes/rx160/visual/link_1.stl"/>
-        </geometry>
-        <xacro:material_staubli_ral_melon_yellow />
-      </visual>
-      <collision>
-        <origin xyz="0 0 0" rpy="0 0 0"/>
-        <geometry>
-          <mesh filename="package://staubli_rx160_support/meshes/rx160/collision/link_1.stl"/>
-        </geometry>
-      </collision>
-      <inertial>
-          <mass value="45.357763"/>
-          <origin xyz="0.085479 -0.002547 -0.040488" rpy="0.0 0.0 0.0"/>
-          <inertia ixx="0.839141" ixy="0.022637" ixz="0.162457"
-                                  iyy="1.030146" iyz="0.027416"
-                                                 izz="1.064698"/>
+        <origin xyz="0 0 0" rpy="0 0 0" />
+        <geometry>
+          <mesh filename="package://staubli_rx160_support/meshes/rx160/visual/link_1.stl" />
+        </geometry>
+        <xacro:material_staubli_ral_melon_yellow />
+      </visual>
+      <collision>
+        <origin xyz="0 0 0" rpy="0 0 0" />
+        <geometry>
+          <mesh filename="package://staubli_rx160_support/meshes/rx160/collision/link_1.stl" />
+        </geometry>
+      </collision>
+      <inertial>
+        <mass value="45.357763" />
+        <origin xyz="0.085479 -0.002547 -0.040488" rpy="0.0 0.0 0.0" />
+        <inertia ixx="0.839141" ixy="0.022637" ixz="0.162457" iyy="1.030146" iyz="0.027416" izz="1.064698" />
       </inertial>
     </link>
     <link name="${prefix}link_2">
       <visual>
-        <origin xyz="0 0 0" rpy="0 0 0"/>
-        <geometry>
-          <mesh filename="package://staubli_rx160_support/meshes/rx160/visual/link_2.stl"/>
-        </geometry>
-        <xacro:material_staubli_ral_melon_yellow />
-      </visual>
-      <collision>
-        <origin xyz="0 0 0" rpy="0 0 0"/>
-        <geometry>
-          <mesh filename="package://staubli_rx160_support/meshes/rx160/collision/link_2.stl"/>
-        </geometry>
-      </collision>
-      <inertial>
-          <mass value="51.266495"/>
-          <origin xyz="-0.000002 0.264164 0.347704" rpy="0.0 0.0 0.0"/>
-          <inertia ixx="5.272800" ixy="0.000010" ixz="0.000017"
-                                  iyy="5.536809" iyz="-0.008261"
-                                                 izz="0.486191"/>
+        <origin xyz="0 0 0" rpy="0 0 0" />
+        <geometry>
+          <mesh filename="package://staubli_rx160_support/meshes/rx160/visual/link_2.stl" />
+        </geometry>
+        <xacro:material_staubli_ral_melon_yellow />
+      </visual>
+      <collision>
+        <origin xyz="0 0 0" rpy="0 0 0" />
+        <geometry>
+          <mesh filename="package://staubli_rx160_support/meshes/rx160/collision/link_2.stl" />
+        </geometry>
+      </collision>
+      <inertial>
+        <mass value="51.266495" />
+        <origin xyz="-0.000002 0.264164 0.347704" rpy="0.0 0.0 0.0" />
+        <inertia ixx="5.272800" ixy="0.000010" ixz="0.000017" iyy="5.536809" iyz="-0.008261" izz="0.486191" />
       </inertial>
     </link>
     <link name="${prefix}link_3">
       <visual>
-        <origin xyz="0 0 0" rpy="0 0 0"/>
-        <geometry>
-          <mesh filename="package://staubli_rx160_support/meshes/rx160/visual/link_3.stl"/>
-        </geometry>
-        <xacro:material_staubli_ral_melon_yellow />
-      </visual>
-      <collision>
-        <origin xyz="0 0 0" rpy="0 0 0"/>
-        <geometry>
-          <mesh filename="package://staubli_rx160_support/meshes/rx160/collision/link_3.stl"/>
-        </geometry>
-      </collision>
-      <inertial>
-          <mass value="19.754401"/>
-          <origin xyz="-0.000255 0.016478 -0.003819" rpy="0.0 0.0 0.0"/>
-          <inertia ixx="0.249388" ixy="-0.004901" ixz="0.004825"
-                                  iyy="0.211780"  iyz="0.000574"
-                                                  izz="0.238488"/>
+        <origin xyz="0 0 0" rpy="0 0 0" />
+        <geometry>
+          <mesh filename="package://staubli_rx160_support/meshes/rx160/visual/link_3.stl" />
+        </geometry>
+        <xacro:material_staubli_ral_melon_yellow />
+      </visual>
+      <collision>
+        <origin xyz="0 0 0" rpy="0 0 0" />
+        <geometry>
+          <mesh filename="package://staubli_rx160_support/meshes/rx160/collision/link_3.stl" />
+        </geometry>
+      </collision>
+      <inertial>
+        <mass value="19.754401" />
+        <origin xyz="-0.000255 0.016478 -0.003819" rpy="0.0 0.0 0.0" />
+        <inertia ixx="0.249388" ixy="-0.004901" ixz="0.004825" iyy="0.211780" iyz="0.000574" izz="0.238488" />
       </inertial>
     </link>
     <link name="${prefix}link_4">
       <visual>
-        <origin xyz="0 0 0" rpy="0 0 0"/>
-        <geometry>
-          <mesh filename="package://staubli_rx160_support/meshes/rx160/visual/link_4.stl"/>
-        </geometry>
-        <xacro:material_staubli_ral_melon_yellow />
-      </visual>
-      <collision>
-        <origin xyz="0 0 0" rpy="0 0 0"/>
-        <geometry>
-          <mesh filename="package://staubli_rx160_support/meshes/rx160/collision/link_4.stl"/>
-        </geometry>
-      </collision>
-      <inertial>
-          <mass value="15.287896"/>
-          <origin xyz="-0.015515 0.000164 0.340348" rpy="0.0 0.0 0.0"/>
-          <inertia ixx="0.331593" ixy="0.000055" ixz="-0.010688"
-                                  iyy="0.320895" iyz="0.000058"
-                                                 izz="0.086557"/>
+        <origin xyz="0 0 0" rpy="0 0 0" />
+        <geometry>
+          <mesh filename="package://staubli_rx160_support/meshes/rx160/visual/link_4.stl" />
+        </geometry>
+        <xacro:material_staubli_ral_melon_yellow />
+      </visual>
+      <collision>
+        <origin xyz="0 0 0" rpy="0 0 0" />
+        <geometry>
+          <mesh filename="package://staubli_rx160_support/meshes/rx160/collision/link_4.stl" />
+        </geometry>
+      </collision>
+      <inertial>
+        <mass value="15.287896" />
+        <origin xyz="-0.015515 0.000164 0.340348" rpy="0.0 0.0 0.0" />
+        <inertia ixx="0.331593" ixy="0.000055" ixz="-0.010688" iyy="0.320895" iyz="0.000058" izz="0.086557" />
       </inertial>
     </link>
     <link name="${prefix}link_5">
       <visual>
-        <origin xyz="0 0 0" rpy="0 0 0"/>
-        <geometry>
-          <mesh filename="package://staubli_rx160_support/meshes/rx160/visual/link_5.stl"/>
+        <origin xyz="0 0 0" rpy="0 0 0" />
+        <geometry>
+          <mesh filename="package://staubli_rx160_support/meshes/rx160/visual/link_5.stl" />
         </geometry>
         <xacro:material_staubli_ral_grey_aluminium />
       </visual>
       <collision>
-        <origin xyz="0 0 0" rpy="0 0 0"/>
-        <geometry>
-          <mesh filename="package://staubli_rx160_support/meshes/rx160/collision/link_5.stl"/>
-        </geometry>
-      </collision>
-      <inertial>
-          <mass value="0.548088"/>
-          <origin xyz="0.000000 -0.000347 0.023671" rpy="0.0 0.0 0.0"/>
-          <inertia ixx="0.000876" ixy="0.000000" ixz="0.000000"
-                                  iyy="0.000889" iyz="0.000005"
-                                                 izz="0.000412"/>
+        <origin xyz="0 0 0" rpy="0 0 0" />
+        <geometry>
+          <mesh filename="package://staubli_rx160_support/meshes/rx160/collision/link_5.stl" />
+        </geometry>
+      </collision>
+      <inertial>
+        <mass value="0.548088" />
+        <origin xyz="0.000000 -0.000347 0.023671" rpy="0.0 0.0 0.0" />
+        <inertia ixx="0.000876" ixy="0.000000" ixz="0.000000" iyy="0.000889" iyz="0.000005" izz="0.000412" />
       </inertial>
     </link>
     <link name="${prefix}link_6">
       <visual>
-        <origin xyz="0 0 0" rpy="0 0 0"/>
-        <geometry>
-          <mesh filename="package://staubli_rx160_support/meshes/rx160/visual/link_6.stl"/>
+        <origin xyz="0 0 0" rpy="0 0 0" />
+        <geometry>
+          <mesh filename="package://staubli_rx160_support/meshes/rx160/visual/link_6.stl" />
         </geometry>
         <xacro:material_staubli_ral_grey_aluminium />
       </visual>
       <collision>
-        <origin xyz="0 0 0" rpy="0 0 0"/>
-        <geometry>
-          <mesh filename="package://staubli_rx160_support/meshes/rx160/collision/link_6.stl"/>
-        </geometry>
-      </collision>
-      <inertial>
-          <mass value="0.038484"/>
-          <origin xyz="-0.000245 0.000000 -0.007626" rpy="0.0 0.0 0.0"/>
-          <inertia ixx="0.000011" ixy="0.000000" ixz="0.000000"
-                                  iyy="0.000011" iyz="0.000000"
-                                                 izz="0.000021"/>
+        <origin xyz="0 0 0" rpy="0 0 0" />
+        <geometry>
+          <mesh filename="package://staubli_rx160_support/meshes/rx160/collision/link_6.stl" />
+        </geometry>
+      </collision>
+      <inertial>
+        <mass value="0.038484" />
+        <origin xyz="-0.000245 0.000000 -0.007626" rpy="0.0 0.0 0.0" />
+        <inertia ixx="0.000011" ixy="0.000000" ixz="0.000000" iyy="0.000011" iyz="0.000000" izz="0.000021" />
       </inertial>
     </link>
     <!-- joints: main serial chain -->
     <joint name="${prefix}joint_1" type="revolute">
-      <origin xyz="0 0 0.55" rpy="0 0 0"/>
-      <parent link="${prefix}base_link"/>
-      <child link="${prefix}link_1"/>
-      <axis xyz="0 0 1"/>
+      <origin xyz="0 0 0.55" rpy="0 0 0" />
+      <parent link="${prefix}base_link" />
+      <child link="${prefix}link_1" />
+      <axis xyz="0 0 1" />
       <limit lower="${radians(-160)}" upper="${radians(160)}" effort="692.0" velocity="${radians(200)}" />
-      <dynamics damping="0.0" friction="0.0"/>
+      <dynamics damping="0.0" friction="0.0" />
     </joint>
     <joint name="${prefix}joint_2" type="revolute">
-      <origin xyz="0.15 0 0" rpy="0 0 0"/>
-      <parent link="${prefix}link_1"/>
-      <child link="${prefix}link_2"/>
-      <axis xyz="0 1 0"/>
+      <origin xyz="0.15 0 0" rpy="0 0 0" />
+      <parent link="${prefix}link_1" />
+      <child link="${prefix}link_2" />
+      <axis xyz="0 1 0" />
       <limit lower="${radians(-137.5)}" upper="${radians(137.5)}" effort="574.0" velocity="${radians(200)}" />
-      <dynamics damping="0.0" friction="0.0"/>
+      <dynamics damping="0.0" friction="0.0" />
     </joint>
     <joint name="${prefix}joint_3" type="revolute">
-      <origin xyz="0 0 0.825" rpy="0 0 0"/>
-      <parent link="${prefix}link_2"/>
-      <child link="${prefix}link_3"/>
-      <axis xyz="0 1 0"/>
+      <origin xyz="0 0 0.825" rpy="0 0 0" />
+      <parent link="${prefix}link_2" />
+      <child link="${prefix}link_3" />
+      <axis xyz="0 1 0" />
       <limit lower="${radians(-150)}" upper="${radians(150)}" effort="242.0" velocity="${radians(255)}" />
-      <dynamics damping="0.0" friction="0.0"/>
+      <dynamics damping="0.0" friction="0.0" />
     </joint>
     <joint name="${prefix}joint_4" type="revolute">
-      <origin xyz="0 0 0" rpy="0 0 0"/>
-      <parent link="${prefix}link_3"/>
-      <child link="${prefix}link_4"/>
-      <axis xyz="0 0 1"/>
+      <origin xyz="0 0 0" rpy="0 0 0" />
+      <parent link="${prefix}link_3" />
+      <child link="${prefix}link_4" />
+      <axis xyz="0 0 1" />
       <limit lower="${radians(-270)}" upper="${radians(270)}" effort="58.0" velocity="${radians(315)}" />
-      <dynamics damping="0.0" friction="0.0"/>
+      <dynamics damping="0.0" friction="0.0" />
     </joint>
     <joint name="${prefix}joint_5" type="revolute">
-      <origin xyz="0 0 0.625" rpy="0 0 0"/>
-      <parent link="${prefix}link_4"/>
-      <child link="${prefix}link_5"/>
-      <axis xyz="0 1 0"/>
+      <origin xyz="0 0 0.625" rpy="0 0 0" />
+      <parent link="${prefix}link_4" />
+      <child link="${prefix}link_5" />
+      <axis xyz="0 1 0" />
       <!-- from Staubli instruction manual:
       (1) effort limit = 58 Nm if axis 6 torque = 0 Nm
       (2) effort limit = 29 Nm for maximum torque on axis 6 -->
       <limit lower="${radians(-105)}" upper="${radians(120)}" effort="29.0" velocity="${radians(360)}" />
-      <dynamics damping="0.0" friction="0.0"/>
+      <dynamics damping="0.0" friction="0.0" />
     </joint>
     <joint name="${prefix}joint_6" type="revolute">
-      <origin xyz="0 0 0.11" rpy="0 0 0"/>
-      <parent link="${prefix}link_5"/>
-      <child link="${prefix}link_6"/>
-      <axis xyz="0 0 1"/>
+      <origin xyz="0 0 0.11" rpy="0 0 0" />
+      <parent link="${prefix}link_5" />
+      <child link="${prefix}link_6" />
+      <axis xyz="0 0 1" />
       <limit lower="${radians(-270)}" upper="${radians(270)}" effort="29.0" velocity="${radians(870)}" />
-      <dynamics damping="0.0" friction="0.0"/>
+      <dynamics damping="0.0" friction="0.0" />
     </joint>
     <!-- ROS-Industrial 'base' frame: base_link to Staubli World Coordinates transform -->
     <link name="${prefix}base" />
     <joint name="${prefix}base_link-base" type="fixed">
-      <origin xyz="0 0 0.550" rpy="0 0 0"/>
-      <parent link="${prefix}base_link"/>
-      <child link="${prefix}base"/>
+      <origin xyz="0 0 0.550" rpy="0 0 0" />
+      <parent link="${prefix}base_link" />
+      <child link="${prefix}base" />
     </joint>
     <!-- ROS-Industrial 'flange' frame: attachment point for EEF models -->
