Commit message: rx160 trouble

File: staubli_rx160_gazebo/urdf/rx160.xacro (robot description, xacro)
@@ -1,12 +1,18 @@
-<?xml version="1.0" ?>
+<?xml version="1.0"?>
 <robot name="staubli_rx160_gazebo" xmlns:xacro="http://wiki.ros.org/xacro">
-  <!-- RX160 -->
-  <xacro:include filename="$(find staubli_rx160_gazebo)/urdf/rx160_macro.xacro"/>
-  <xacro:staubli_rx160_robot prefix=""/>
+  <!-- TX60 -->
+  <xacro:include filename="$(find staubli_rx160_gazebo)/urdf/rx160_macro.xacro" />
+  <xacro:include filename="$(find staubli_rx160_gazebo)/urdf/_d435.urdf.xacro" />
+  <xacro:include filename="$(find staubli_rx160_support)/urdf/gripper_macro.xacro" />
+  <xacro:staubli_rx160_robot prefix="" />
+  <xacro:gripper prefix="" />
+  <sensor_d435 parent="link_6">
+    <origin xyz="0.105 -0.0 0.01" rpy="0 -1.57 3.14" />
+  </sensor_d435>
   <!-- Fix robot to Gazebo world -->
-  <link name="world"/>
+  <link name="world" />
   <joint name="world-base_link-fixed" type="fixed">
-    <parent link="world"/>
-    <child link="base_link"/>
+    <parent link="world" />
+    <child link="base_link" />
     <origin xyz="0.0 0.0 0.0" rpy="0.0 0.0 0.0" />
   </joint>

File: staubli_rx160_gazebo/urdf/rx160_macro.xacro (robot description, xacro)
@@ -1,106 +1,106 @@
 <?xml version="1.0"?>
 <robot xmlns:xacro="http://wiki.ros.org/xacro">
-<xacro:include filename="$(find staubli_rx160_support)/urdf/rx160_macro.xacro"/>
-<xacro:macro name="staubli_rx160_robot" params="prefix">
-  <!-- get URDF description of Staubli RX160 model -->
-  <xacro:staubli_rx160 prefix="${prefix}" />
-  <!-- transmission list -->
-  <transmission name="${prefix}tran1">
-    <robotNamespace>/${prefix}</robotNamespace>
-    <type>transmission_interface/SimpleTransmission</type>
-    <joint name="${prefix}joint_1">
-      <hardwareInterface>hardware_interface/PositionJointInterface</hardwareInterface>
-    </joint>
-    <actuator name="${prefix}motor1">
-      <mechanicalReduction>1</mechanicalReduction>
-    </actuator>
-  </transmission>
-  <transmission name="${prefix}tran2">
-    <robotNamespace>/${prefix}</robotNamespace>
-    <type>transmission_interface/SimpleTransmission</type>
-    <joint name="${prefix}joint_2">
-      <hardwareInterface>hardware_interface/PositionJointInterface</hardwareInterface>
-    </joint>
-    <actuator name="${prefix}motor2">
-      <mechanicalReduction>1</mechanicalReduction>
-    </actuator>
-  </transmission>
-  <transmission name="${prefix}tran3">
-    <robotNamespace>/${prefix}</robotNamespace>
-    <type>transmission_interface/SimpleTransmission</type>
-    <joint name="${prefix}joint_3">
-      <hardwareInterface>hardware_interface/PositionJointInterface</hardwareInterface>
-    </joint>
-    <actuator name="${prefix}motor3">
-      <mechanicalReduction>1</mechanicalReduction>
-    </actuator>
-  </transmission>
-  <transmission name="${prefix}tran4">
-    <robotNamespace>/${prefix}</robotNamespace>
-    <type>transmission_interface/SimpleTransmission</type>
-    <joint name="${prefix}joint_4">
-      <hardwareInterface>hardware_interface/PositionJointInterface</hardwareInterface>
-    </joint>
-    <actuator name="${prefix}motor4">
-      <mechanicalReduction>1</mechanicalReduction>
-    </actuator>
-  </transmission>
-  <transmission name="${prefix}tran5">
-    <robotNamespace>/${prefix}</robotNamespace>
-    <type>transmission_interface/SimpleTransmission</type>
-    <joint name="${prefix}joint_5">
-      <hardwareInterface>hardware_interface/PositionJointInterface</hardwareInterface>
-    </joint>
-    <actuator name="${prefix}motor5">
-      <mechanicalReduction>1</mechanicalReduction>
-    </actuator>
-  </transmission>
-  <transmission name="${prefix}tran6">
-    <robotNamespace>/${prefix}</robotNamespace>
-    <type>transmission_interface/SimpleTransmission</type>
-    <joint name="${prefix}joint_6">
-      <hardwareInterface>hardware_interface/PositionJointInterface</hardwareInterface>
-    </joint>
-    <actuator name="${prefix}motor6">
-      <mechanicalReduction>1</mechanicalReduction>
-    </actuator>
-  </transmission>
-  <!-- end of transmission list -->
-  <!-- Gazebo-specific link properties -->
-  <gazebo reference="${prefix}base_link">
-    <material>Gazebo/Yellow</material>
-    <turnGravityOff>true</turnGravityOff>
-  </gazebo>
-  <gazebo reference="${prefix}link_1">
-    <material>Gazebo/Yellow</material>
-    <turnGravityOff>true</turnGravityOff>
-  </gazebo>
-  <gazebo reference="${prefix}link_2">
-    <material>Gazebo/Yellow</material>
-    <turnGravityOff>true</turnGravityOff>
-  </gazebo>
-  <gazebo reference="${prefix}link_3">
-    <material>Gazebo/Yellow</material>
-    <turnGravityOff>true</turnGravityOff>
-  </gazebo>
-  <gazebo reference="${prefix}link_4">
-    <material>Gazebo/Yellow</material>
-    <turnGravityOff>true</turnGravityOff>
-  </gazebo>
-  <gazebo reference="${prefix}link_5">
-    <material>Gazebo/Grey</material>
-    <turnGravityOff>true</turnGravityOff>
-  </gazebo>
-  <gazebo reference="${prefix}link_6">
-    <material>Gazebo/Grey</material>
-    <turnGravityOff>true</turnGravityOff>
-  </gazebo>
-  <!-- ros_control plugin -->
-  <gazebo>
-    <plugin name="gazebo_ros_control" filename="libgazebo_ros_control.so">
+  <xacro:include filename="$(find staubli_rx160_support)/urdf/rx160_macro.xacro" />
+  <xacro:macro name="staubli_rx160_robot" params="prefix">
+    <!-- get URDF description of Staubli TX60 model -->
+    <xacro:staubli_rx160 prefix="${prefix}" />
+    <!-- transmission list -->
+    <transmission name="${prefix}tran1">
       <robotNamespace>/${prefix}</robotNamespace>
-      <robotSimType>gazebo_ros_control/DefaultRobotHWSim</robotSimType>
-    </plugin>
-  </gazebo>
+      <type>transmission_interface/SimpleTransmission</type>
+      <joint name="${prefix}joint_1">
+        <hardwareInterface>hardware_interface/PositionJointInterface</hardwareInterface>
+      </joint>
+      <actuator name="${prefix}motor1">
+        <mechanicalReduction>1</mechanicalReduction>
+      </actuator>
+    </transmission>
+    <transmission name="${prefix}tran2">
+      <robotNamespace>/${prefix}</robotNamespace>
+      <type>transmission_interface/SimpleTransmission</type>
+      <joint name="${prefix}joint_2">
+        <hardwareInterface>hardware_interface/PositionJointInterface</hardwareInterface>
+      </joint>
+      <actuator name="${prefix}motor2">
+        <mechanicalReduction>1</mechanicalReduction>
+      </actuator>
+    </transmission>
+    <transmission name="${prefix}tran3">
+      <robotNamespace>/${prefix}</robotNamespace>
+      <type>transmission_interface/SimpleTransmission</type>
+      <joint name="${prefix}joint_3">
+        <hardwareInterface>hardware_interface/PositionJointInterface</hardwareInterface>
+      </joint>
+      <actuator name="${prefix}motor3">
+        <mechanicalReduction>1</mechanicalReduction>
+      </actuator>
+    </transmission>
+    <transmission name="${prefix}tran4">
+      <robotNamespace>/${prefix}</robotNamespace>
+      <type>transmission_interface/SimpleTransmission</type>
+      <joint name="${prefix}joint_4">
+        <hardwareInterface>hardware_interface/PositionJointInterface</hardwareInterface>
+      </joint>
+      <actuator name="${prefix}motor4">
+        <mechanicalReduction>1</mechanicalReduction>
+      </actuator>
+    </transmission>
+    <transmission name="${prefix}tran5">
+      <robotNamespace>/${prefix}</robotNamespace>
+      <type>transmission_interface/SimpleTransmission</type>
+      <joint name="${prefix}joint_5">
+        <hardwareInterface>hardware_interface/PositionJointInterface</hardwareInterface>
+      </joint>
+      <actuator name="${prefix}motor5">
+        <mechanicalReduction>1</mechanicalReduction>
+      </actuator>
+    </transmission>
+    <transmission name="${prefix}tran6">
+      <robotNamespace>/${prefix}</robotNamespace>
+      <type>transmission_interface/SimpleTransmission</type>
+      <joint name="${prefix}joint_6">
+        <hardwareInterface>hardware_interface/PositionJointInterface</hardwareInterface>
+      </joint>
+      <actuator name="${prefix}motor6">
+        <mechanicalReduction>1</mechanicalReduction>
+      </actuator>
+    </transmission>
+    <!-- end of transmission list -->
+    <!-- Gazebo-specific link properties -->
+    <gazebo reference="${prefix}base_link">
+      <material>Gazebo/Yellow</material>
+      <turnGravityOff>true</turnGravityOff>
+    </gazebo>
+    <gazebo reference="${prefix}link_1">
+      <material>Gazebo/Yellow</material>
+      <turnGravityOff>true</turnGravityOff>
+    </gazebo>
+    <gazebo reference="${prefix}link_2">
+      <material>Gazebo/Yellow</material>
+      <turnGravityOff>true</turnGravityOff>
+    </gazebo>
+    <gazebo reference="${prefix}link_3">
+      <material>Gazebo/Yellow</material>
+      <turnGravityOff>true</turnGravityOff>
+    </gazebo>
+    <gazebo reference="${prefix}link_4">
+      <material>Gazebo/Yellow</material>
+      <turnGravityOff>true</turnGravityOff>
+    </gazebo>
+    <gazebo reference="${prefix}link_5">
+      <material>Gazebo/Grey</material>
+      <turnGravityOff>true</turnGravityOff>
+    </gazebo>
+    <gazebo reference="${prefix}link_6">
+      <material>Gazebo/Grey</material>
+      <turnGravityOff>true</turnGravityOff>
+    </gazebo>
+    <!-- ros_control plugin -->
+    <gazebo>
+      <plugin name="gazebo_ros_control" filename="libgazebo_ros_control.so">
+        <robotNamespace>/${prefix}</robotNamespace>
+        <robotSimType>gazebo_ros_control/DefaultRobotHWSim</robotSimType>
+      </plugin>
+    </gazebo>
   </xacro:macro>
 </robot>
