Commit message: tx200 not working

File: staubli_tx200_support/urdf/tx200_macro.xacro (robot description, xacro)
@@ -108,5 +108,5 @@
         <origin xyz="0 0 0" rpy="0 0 0" />
         <geometry>
-          <mesh filename="package://staubli_tx60_support/meshes/tx60/visual/link_5.stl" />
+          <mesh filename="package://staubli_tx200_support/meshes/tx200/visual/link_5.stl" />
         </geometry>
         <xacro:material_staubli_ral_grey_aluminium />
@@ -115,5 +115,5 @@
         <origin xyz="0 0 0" rpy="0 0 0" />
         <geometry>
-          <mesh filename="package://staubli_tx60_support/meshes/tx60/collision/link_5.stl" />
+          <mesh filename="package://staubli_tx200_support/meshes/tx200/collision/link_5.stl" />
         </geometry>
       </collision>
@@ -128,5 +128,5 @@
         <origin xyz="0 0 0" rpy="0 0 0" />
         <geometry>
-          <mesh filename="package://staubli_tx60_support/meshes/tx60/visual/link_6.stl" />
+          <mesh filename="package://staubli_tx200_support/meshes/tx200/visual/link_6.stl" />
         </geometry>
         <xacro:material_staubli_ral_grey_aluminium />
@@ -135,5 +135,5 @@
         <origin xyz="0 0 0" rpy="0 0 0" />
         <geometry>
-          <mesh filename="package://staubli_tx60_support/meshes/tx60/collision/link_6.stl" />
+          <mesh filename="package://staubli_tx200_support/meshes/tx200/collision/link_6.stl" />
         </geometry>
       </collision>
